File: Breakout/Soap/Soap.sch (EAGLE design)
At the start: 23 parts, among them U2 MCP73831

Commit message: switch charger
Parts:
- removed C3, C6: 4.7uF, SparkFun-Capacitors:CAP0603-CAP
- removed C4, C5: 22uF, rcl:C-EUC0603
- removed C7: 0.1uF, adafruit:C-USC0402
- removed D3: BAT20J, SparkFun-DiscreteSemi:DIODE-SCHOTTKY-BAT20J
- removed JP2: USB-RECEPTABLE-HIROSE-ZX62-AB-5PA(11), daspilker:USB-RECEPTABLE-HIROSE-ZX62-AB-5PA(11)
- removed L1: 2.2uH, Spark:INDUCTOR-SPARKFUN0805
- removed LED1, LED2: (no value), eagle-ltspice:LED_E
- removed LMR: MCP1824T-3302E/OT, Microchip_By_element14_Batch_1:MCP1824T-3302E/OT
- removed R2: 10K 1%, SparkFun-Resistors:RESISTOR0603
- removed R3, R6: 470-Ohm, SparkFun-Resistors:RESISTOR0603
- removed R4: 100K, adafruit:R-US_R0402
- removed R5: 2K, SparkFun-Resistors:RESISTOR0603
- removed U2: MCP73831, BaseApp:MCP73831
- added C12, C8: 10uF, rcl:C-EUC0603
- added CHARG/LBO: ORANGE, led:LEDSML0603
- added DONE: GREEN, led:LEDSML0603
- added L2: 2.2uH, SparkFun-Passives:INDUCTOR0805
- added PWR: RED, led:LEDSML0603
- added R10: 100K, SparkFun-Passives:RESISTOR0603-RES
- added R11, R12, R13, R14, R15: 1K, SparkFun-Passives:RESISTOR0603-RES
- added R7: 100K, SparkFun-Resistors:RESISTOR0603
- added R9: 2K, SparkFun-Passives:RESISTOR0603-RES
- added THERMAL: 10K, SparkFun-Passives:RESISTOR0603-RES
- added U$2: MCP73871-2CCI/ML, microchip-battery:MCP73871-2CCI/ML
- added U1: TPS63001DRCT, TPS63001:TPS63001DRCT
- added USB: MICRO-USB-ZX62R-B-5P, con-hirose:MICRO-USB-ZX62R-B-5P
- R1: value 45.2k 1% -> 470K
Connections:
- removed net FB: LMR.FB, R1.1, R2.2
- removed net N$1: LED2.A, R3.2
- removed net N$2: LMR.EN, R4.1
- removed net N$3: R5.2, U2.PROG
- removed net N$5: LED1.C, R6.2
- removed net STAT: LED1.A, LED2.C, U2.STAT
- removed net SW: D3.C, L1.1, LMR.SW
- removed net VBAT: C3.1, C4.1, J1.+, LMR.VIN, R4.2, U2.VBAT
- removed net VIN: C6.1, JP2.VCC, R3.1, U2.VDD
- new net +5V_USB: R11.2, R12.2, R13.2, R14.2, U$2./TE, U$2.CE, U$2.IN, U$2.IN2, U$2.PROG2, U$2.SEL, USB.1
- new net +BATT: J1.+, R1.2, U$2.VBAT, U$2.VBAT2, U$2.VBAT_SENSE
- new net GPIO_05: R1.1, R7.2
- new net N$52: L2.1, U1.L1
- new net N$53: L2.2, U1.L2
- new net N$55: R9.2, U$2.PROG3
- new net N$56: R10.2, U$2.PROG1
- new net N$57: PWR.A, U$2./PG
- new net N$58: DONE.A, U$2.STAT2
- new net N$59: CHARG/LBO.A, U$2.STAT1/LBO
- new net N$60: CHARG/LBO.C, R11.1
- new net N$61: DONE.C, R12.1
- new net N$62: PWR.C, R13.1
- new net N$63: R14.1, R15.2, U$2.VPCC
- new net N$64: THERMAL.2, U$2.THERM
- new net OUT: C12.1, U$2.OUT, U$2.OUT2, U1.EN, U1.PS/SYNC, U1.VIN, U1.VINA
- new net VCC: C8.1, U1.FB, U1.VOUT
- net +3V3: no longer C5.1, C7.1, L1.2, R1.2
- net GND: now also C12.2, C8.2, R10.1, R15.1, R7.1, R9.1, THERMAL.1, U$2.EP, U$2.VSS, U$2.VSS2, U1.GND, U1.PGND, U1.POWER_PAD, USB.5; no longer C3.2, C4.2, C5.2, C6.2, C7.2, D3.A, JP2.GND, LMR.GND, R2.1, R5.1, R6.1, U2.VSS
Other:
- note added: "+5V_CHARGE"
- note added: "3.3V"
- note added: "BATT"
- note added: "GND"
- note added: "LIPO Charger with USB"
- note added: "Optional"
- note added: "Voltage Regulator"
