File: Breakout/breakout.sch (EAGLE design)
At the start: 27 parts, among them U1 TPS63001DRCT, U2 MCP73831

Commit message: Add Bom file
Parts:
- C1: value (none) -> 1pF
- L1: value (none) -> 3.6nH
Changed lines of the file:
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@@
 <part name="CC3200MOD" library="cc3200mod" deviceset="CC3200" device=""/>
 <part name="ANT_PAD" library="Antenna" deviceset="ANT" device=""/>
-<part name="C1" library="rcl" deviceset="C-US" device="C0402"/>
-<part name="L1" library="Spark" deviceset="INDUCTOR-SPARKFUN" device="0402"/>
+<part name="C1" library="rcl" deviceset="C-US" device="C0402" value="1pF"/>
+<part name="L1" library="Spark" deviceset="INDUCTOR-SPARKFUN" device="0402" value="3.6nH"/>
 <part name="JTAG" library="con-lstb" deviceset="MA06-1" device=""/>
 <part name="U$1" library="LaunchPadXL" deviceset="XL" device=""/>

Commit message: switch charger
Parts:
- removed C2, C3: 4.7uF, rcl:C-EUC0603
- removed CHARGING, FULL: (no value), eagle-ltspice:LED_ESML0603
- removed R1, R4: 470 Ohm, SparkFun-Resistors:RESISTOR0603
- removed R2: 2 k, SparkFun-Resistors:RESISTOR0603
- removed R5, R6: 100K, SparkFun-Resistors:RESISTOR0603
- removed U2: MCP73831, BaseApp:MCP73831
- added CHARG/LBO: ORANGE, led:LEDSML0603
- added DONE: GREEN, led:LEDSML0603
- added PWR: RED, led:LEDSML0603
- added R10: 100K, SparkFun-Passives:RESISTOR0603-RES
- added R11, R12, R13, R14, R15: 1K, SparkFun-Passives:RESISTOR0603-RES
- added R9: 2K, SparkFun-Passives:RESISTOR0603-RES
- added THERMAL: 10K, SparkFun-Passives:RESISTOR0603-RES
- added U$2: MCP73871-2CCI/ML, microchip-battery:MCP73871-2CCI/ML
- renumbered U$1 to U11
Connections:
- removed net +5V_CHARGE: C2.1, CHARGING.A, U2.VDD, USB.1
- removed net N$7: CHARGING.C, R1.2
- removed net PROG: R2.2, U2.PROG
- removed net STAT: R1.1, R4.1, R6.1, U2.STAT
- new net +5V_USB: R11.2, R12.2, R13.2, R14.2, U$2./TE, U$2.CE, U$2.IN, U$2.IN2, U$2.PROG2, U$2.SEL, USB.1
- new net N$17: R9.2, U$2.PROG3
- new net N$20: R10.2, U$2.PROG1
- new net N$26: PWR.A, U$2./PG
- new net N$31: DONE.A, U$2.STAT2
- new net N$32: CHARG/LBO.A, U$2.STAT1/LBO
- new net N$33: CHARG/LBO.C, R11.1
- new net N$35: DONE.C, R12.1
- new net N$36: PWR.C, R13.1
- new net N$37: R14.1, R15.2, U$2.VPCC
- new net OUT: C12.1, U$2.OUT, U$2.OUT2, U1.EN, U1.PS/SYNC, U1.VIN, U1.VINA
- net +BATT: now also U$2.VBAT, U$2.VBAT2, U$2.VBAT_SENSE; no longer C12.1, C3.1, U1.EN, U1.PS/SYNC, U1.VIN, U1.VINA, U2.VBAT
- net GND: now also R10.1, R15.1, R9.1, THERMAL.1, U$2.EP, U$2.VSS, U$2.VSS2; no longer C2.2, C3.2, FULL.C, R2.1, R5.2, U2.VSS
- net GPIO_22: no longer R5.1, R6.2
- net N$28: now also THERMAL.2, U$2.THERM; no longer FULL.A, R4.2

Commit message: Added FTDI reroute
Parts:
- removed FLASH, JTAG: (no value), con-lstb:MA06-1
- added C2, C3: 27pF, SparkFun-Passives:CAP0402-CAP
- added C4: 33nF, SparkFun-Passives:CAP0402-CAP
- added C5: 0.1uF, SparkFun-Passives:CAP0402-CAP
- added Q1: 16Mhz, crystal:CRYSTALTC26H
- added R1: 1.5K, SparkFun-Resistors:RESISTOR0603
- added R16, R17, R18, R19, R21, R22, R24, R5, R6: 33, SparkFun-Resistors:RESISTOR0603
- added R2, R4: 28, SparkFun-Passives:RESISTOR0603-RES
- added R20: 10k, SparkFun-Resistors:RESISTOR0603
- added R23: 470, SparkFun-Resistors:RESISTOR0603
- added S1: (no value), Spark:TAC_SWITCHSMD
- added U$1: FT2232D, SparkFun-DigitalIC:FT2232D
- added U$3: DECADE-74LVC125A, DECADE-libraries:DECADE-74LVC125A
Connections:
- removed net JTAG_TCK: CC3200MOD.21_JTAG_TCK, JTAG.5
- removed net JTAG_TMS: CC3200MOD.22_JTAP_TMS, JTAG.6
- removed net RX: CC3200MOD.46_GPIO1, FLASH.4, U11.GPIO_01
- removed net TX: CC3200MOD.47_GPO2, FLASH.5, U11.GPIO_02
- new net DBGEN_N: R18.2, U$3.OE1
- new net DBG_RST_N: R19.2, R20.1, U$3.OE2
- new net FTDI_RX: CC3200MOD.46_GPIO1, R6.2, U11.GPIO_01
- new net FTDI_TX: CC3200MOD.47_GPO2, R5.2, U11.GPIO_02
- new net FT_SK: R17.2, U$3.1A
- new net N$38: C2.2, Q1.2, U$1.XTIN
- new net N$39: USB.4
- new net N$40: C3.2, Q1.1, U$1.XTOUT
- new net N$41: R4.1, USB.3
- new net N$42: R2.1, USB.2
- new net N$43: C4.2, U$1.3V3OUT
- new net N$44: R5.1, U$1.BDBUS0
- new net N$45: R6.1, U$1.BDBUS1
- new net N$46: R17.1, U$1.ADBUS0
- new net N$47: R19.1, U$1.ADBUS5
- new net N$48: R18.1, U$1.ADBUS6
- new net N$49: R21.2, U$3.2A
- new net N$50: R22.2, U$3.2Y
- new net N$51: C5.2, R23.1, U$1.AVCC
- new net N$53: R24.1, S1.3, S1.4
- new net N$7: R1.2, U$1.RSTOUT#
- new net TCK: R16.2, U$3.1Y
- new net USB_DM: R4.2, U$1.USBDM
- new net USB_DP: R1.1, R2.2, U$1.USBDP
- net +5V_USB: now also R23.2, U$1.RESET#, U$1.VCC1, U$1.VCC2
- net GND: now also C2.1, C3.1, C4.1, C5.1, R21.1, R24.2, U$1.AGND, U$1.GND1, U$1.GND2, U$1.GND3, U$1.GND4, U$1.TEST, U$3.GND; no longer FLASH.1, JTAG.1
- net JTAG_TDI: no longer JTAG.3
- net JTAG_TDO: no longer JTAG.4
- net N_RESET: now also R22.1, S1.1, S1.2; no longer FLASH.6
- net SOP2: now also R16.1; no longer FLASH.3
- net VCC: now also R20.2, U$1.VCCIOA, U$1.VCCIOB, U$3.VCC; no longer FLASH.2, JTAG.2
Other:
- note removed: "+5V_CHARGE"
- note removed: "GND"
- note removed: "Optional"
- moved on the sheet: USB
