File: Breakout/breakout.brd (EAGLE design)
At the start: 52.6 x 42.5 mm, 49 parts, among them Q1 16Mhz, U1 TPS63001DRCT, U11 XL

Commit message: Finish un-routed grounds
Parts:
- moved R5 0.82 mm to (18.5, 30.1)
Routing:
- net GND: track 36.9 -> 41.2 mm, vias 42 -> 43
- net FTDI_TX: track 36.0 -> 35.3 mm
- net N$44: track 40.1 -> 39.5 mm
Changed lines of the file:
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@@
 <element name="C4" library="SparkFun-Passives" package="0402-CAP" value="33nF" x="39.8" y="5.62"/>
 <element name="U$3" library="DECADE-libraries" package="DECADE-SO-14" value="DECADE-74LVC125A" x="52.11" y="26.39" rot="R270"/>
-<element name="R5" library="SparkFun-Resistors" package="0603-RES" value="33" x="18.82" y="30.87" rot="R180"/>
+<element name="R5" library="SparkFun-Resistors" package="0603-RES" value="33" x="18.5" y="30.12" rot="R180"/>
 <element name="R6" library="SparkFun-Resistors" package="0603-RES" value="33" x="55.3" y="16.56"/>
 <element name="R16" library="SparkFun-Resistors" package="0603-RES" value="33" x="44.77" y="27.43"/>
@@
 <via x="38.61" y="2.28" extent="1-16" drill="0.4"/>
 <via x="49.16" y="3.16" extent="1-16" drill="0.4"/>
-<wire x1="50.34" y1="15.62" x2="45.84" y2="15.62" width="0" layer="19" extent="1-1"/>
-<wire x1="22.07" y1="30.315" x2="23.5" y2="33.54" width="0" layer="19" extent="1-16"/>
 <wire x1="49.2928" y1="4.19" x2="49.2928" y2="3.2928" width="0.254" layer="1"/>
 <wire x1="49.2928" y1="3.2928" x2="49.16" y2="3.16" width="0.254" layer="1"/>
+<via x="18.45" y="31.19" extent="1-16" drill="0.4"/>
+<wire x1="22.07" y1="30.315" x2="22.04" y2="30.315" width="0.4064" layer="1"/>
+<wire x1="18.45" y1="31.19" x2="19.84" y2="31.19" width="0.254" layer="1"/>
+<wire x1="19.84" y1="31.19" x2="20.31" y2="30.72" width="0.254" layer="1"/>
+<wire x1="20.31" y1="30.72" x2="20.31" y2="30.4" width="0.254" layer="1"/>
+<wire x1="20.31" y1="30.4" x2="20.48" y2="30.23" width="0.254" layer="1"/>
+<wire x1="20.48" y1="30.23" x2="21.985" y2="30.23" width="0.254" layer="1"/>
+<wire x1="21.985" y1="30.23" x2="22.07" y2="30.315" width="0.254" layer="1"/>
+<wire x1="50.34" y1="15.62" x2="45.84" y2="15.62" width="0" layer="19" extent="1-1"/>
 </signal>
 <signal name="N$1">
@@
 <contactref element="THERMAL" pad="2"/>
 <wire x1="28.32" y1="33.125" x2="28.32" y2="31.55" width="0.3048" layer="1"/>
-<wire x1="28.32" y1="31.55" x2="27.93" y2="31.1" width="0.3048" layer="1"/>
-<wire x1="27.93" y1="31.1" x2="21.40146875" y2="31.08923125" width="0.3048" layer="1"/>
-<wire x1="21.40146875" y1="31.08923125" x2="21" y2="31.03" width="0.3048" layer="1"/>
+<wire x1="28.32" y1="31.55" x2="27.92" y2="31.29" width="0.3048" layer="1"/>
+<wire x1="27.92" y1="31.29" x2="21.39146875" y2="31.27923125" width="0.3048" layer="1"/>
+<wire x1="21.39146875" y1="31.27923125" x2="21" y2="31.03" width="0.3048" layer="1"/>
 <wire x1="20.7" y1="31.5" x2="20.7" y2="33.39" width="0.3048" layer="2"/>
 <via x="20.7" y="33.39" extent="1-16" drill="0.5"/>
@@
 <via x="21" y="31.03" extent="1-16" drill="0.5"/>
 <wire x1="21" y1="31.03" x2="21.4007" y2="31.19" width="0.254" layer="1"/>
-<wire x1="21.4007" y1="31.19" x2="21.40146875" y2="31.08923125" width="0.254" layer="1"/>
+<wire x1="21.4007" y1="31.19" x2="21.39146875" y2="31.27923125" width="0.254" layer="1"/>
 </signal>
 <signal name="USB_DP">
@@
 <contactref element="U$1" pad="40"/>
 <contactref element="R5" pad="1"/>
-<wire x1="19.67" y1="30.87" x2="19.66" y2="29.92" width="0.254" layer="1"/>
+<wire x1="19.35" y1="30.12" x2="19.66" y2="29.92" width="0.254" layer="1"/>
 <wire x1="19.66" y1="29.92" x2="19.98" y2="29.6" width="0.254" layer="1"/>
 <wire x1="19.98" y1="29.6" x2="22.76" y2="29.6" width="0.254" layer="1"/>
@@
 <contactref element="CC3200MOD" pad="P47"/>
 <contactref element="U11" pad="GPIO_02"/>
-<wire x1="17.97" y1="30.87" x2="17.78" y2="30.97" width="0.254" layer="1"/>
-<wire x1="17.78" y1="30.97" x2="16.85" y2="30.04" width="0.254" layer="1"/>
+<wire x1="17.65" y1="30.12" x2="17.33" y2="30.1" width="0.254" layer="1"/>
+<wire x1="17.33" y1="30.1" x2="16.85" y2="30.04" width="0.254" layer="1"/>
 <wire x1="16.85" y1="30.04" x2="16.85" y2="23.94" width="0.254" layer="1"/>
 <wire x1="16.85" y1="23.94" x2="17.94" y2="22.85" width="0.254" layer="1"/>
