File: Breakout/BreakoutFTDI_V1/breakout.sch (EAGLE design)
At the start: 56 parts, among them Q1 16Mhz, U1 TPS63001DRCT, U11 XL

Commit message: Added a Ferrite
Parts:
- added L3: (no value), Spark:INDUCTOR-SPARKFUN0603
Connections:
- new net N$15: L3.1, USB.1
- net +5V_USB: now also L3.2; no longer USB.1
Changed lines of the file:
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@@
 <part name="C10" library="SparkFun-Capacitors" deviceset="CAP" device="0402-CAP" value=".1uF"/>
 <part name="R26" library="SparkFun-Resistors" deviceset="RESISTOR" device="0603" value="100K"/>
+<part name="L3" library="Spark" deviceset="INDUCTOR-SPARKFUN" device="0603"/>
 </parts>
 <sheets>
@@
 <attribute name="VALUE" x="223.52" y="375.158" size="1.778" layer="96"/>
 </instance>
+<instance part="L3" gate="G$1" x="48.26" y="340.36" rot="R90"/>
 </instances>
 <busses>
@@
 </segment>
 <segment>
-<pinref part="USB" gate="G$1" pin="1"/>
-<wire x1="35.56" y1="345.44" x2="43.18" y2="345.44" width="0.1524" layer="91"/>
-<label x="43.18" y="345.44" size="1.778" layer="95"/>
-</segment>
-<segment>
 <pinref part="R11" gate="G$1" pin="2"/>
 <wire x1="68.58" y1="490.22" x2="68.58" y2="495.3" width="0.1524" layer="91"/>
@@
 <wire x1="86.36" y1="355.6" x2="99.06" y2="355.6" width="0.1524" layer="91"/>
 </segment>
+<segment>
+<pinref part="L3" gate="G$1" pin="2"/>
+<wire x1="55.88" y1="340.36" x2="58.42" y2="340.36" width="0.1524" layer="91"/>
+<label x="50.8" y="337.82" size="1.778" layer="95"/>
+</segment>
 </net>
 <net name="N$17" class="0">
@@
 </segment>
 </net>
+<net name="N$15" class="0">
+<segment>
+<pinref part="USB" gate="G$1" pin="1"/>
+<wire x1="35.56" y1="345.44" x2="38.1" y2="345.44" width="0.1524" layer="91"/>
+<wire x1="38.1" y1="345.44" x2="38.1" y2="340.36" width="0.1524" layer="91"/>
+<pinref part="L3" gate="G$1" pin="1"/>
+<wire x1="38.1" y1="340.36" x2="40.64" y2="340.36" width="0.1524" layer="91"/>
+</segment>
+</net>
