File: Breakout/WeBee WiFi CC3200MOD/WeBee.brd (EAGLE design)
At the start: 26.1 x 45.4 mm, 25 parts, among them U1 TPS63001DRCT

Commit message: Finished WeBee
Parts:
- removed C12, C8: 10uF, rcl:C0603
- removed J1: (no value), SparkFun-Connectors:JST-2-SMD
- removed L2: 2.2uH, SparkFun-Passives:0805
- removed U1: TPS63001DRCT, TPS63001:SON50P300X300X100-11N
- added C4, C5: 22uF, rcl:C0603
- added C7: 0.1uF, adafruit:C0402
- added D3: BAT20J, SparkFun-DiscreteSemi:SOD-323
- added J2: (no value), SparkFun-Connectors:JST-2-SMD
- added L1: 2.2uH, Spark:0805
- added R16: 10K 1%, SparkFun-Resistors:0603-RES
- added R3: 0, SparkFun-Passives:0603-RES
- added R4: 100K, adafruit:R0402
- added R5: (no value), microbuilder:0402
- added R8: 45.2k 1%, SparkFun-Resistors:0603-RES
- added S1: (no value), Spark:TACTILE_SWITCH_SMD
- added U3: LMR10510XMFE, Microchip_By_element14_Batch_1:SOT95P270X145-5N
- moved R7 3.94 mm to (19.9, 19.0)
- moved R2 3.84 mm to (4.83, 11.7)
- moved R9 3.82 mm to (5.24, 19.3)
- moved R1 3.70 mm to (4.67, 13.8)
- moved R14 3.45 mm to (15.8, 19.1)
- moved R10 3.39 mm to (4.69, 16.4), turned to 90 degrees
- moved R15 2.97 mm to (12.8, 18.1)
- moved JP2 2.79 mm to (24.5, 42.5)
- moved JP1 2.79 mm to (1.65, 4.45)
- moved JP3 2.79 mm to (6.35, 21.8)
- moved U$1 2.29 mm to (13.0, 35.3)
- moved U$3 1.08 mm to (9.08, 14.9)
Connections:
- removed net N$65: L2.1, U1.4
- removed net N$66: L2.2, U1.2
- new net FB: R16.2, R8.1, U3.3
- new net N$1: R5.1, S1.2
- new net N$11: R4.1, U3.4
- new net SW: D3.C, L1.1, U3.1
- net +5V_USB: now also R3.2
- net +BATT: now also J2.2; no longer J1.2
- net GND: now also C4.2, C5.2, C7.2, D3.A, J2.1, R16.1, S1.3, S1.4, U3.2; no longer C12.2, C8.2, J1.1, U1.11, U1.3, U1.9
- net OUT: now also C4.1, R3.1, R4.2, U3.5; no longer C12.1, U1.5, U1.6, U1.7, U1.8
- net VCC: now also C5.1, C7.1, L1.2, R5.2, R8.2; no longer C8.1, U1.1, U1.10
Routing:
- net N$71: track 45.0 -> 14.4 mm, vias 4 -> 2
- net N$70: track 43.2 -> 12.6 mm
- net N$31: track 22.5 -> 39.2 mm, vias 2 -> 1
- net +5V_USB: track 30.8 -> 45.6 mm, vias 3 -> 6
- net N$11: track 0.00 -> 13.1 mm, vias 0 -> 2
- net N$1: track 0.00 -> 11.3 mm
- net SW: track 0.00 -> 10.4 mm
- net GPIO_05: track 29.1 -> 19.7 mm, vias 4 -> 2
- net OUT: track 12.9 -> 21.8 mm, vias 2 -> 4
- net FB: track 0.00 -> 8.66 mm
- net GND: track 101.4 -> 109.9 mm, vias 2 -> 1
- net N$65: track 7.97 -> 0.00 mm, vias 2 -> 0
- net N$77: track 19.6 -> 26.2 mm
- net N$66: track 5.40 -> 0.00 mm, vias 2 -> 0
- net N$72: track 17.8 -> 22.2 mm
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Other:
- board size 26.1 x 45.4 mm -> 26.1 x 47.9 mm
