File: Breakout/WeBee WiFi CC3200MOD/WeBee.sch (EAGLE design)
At the start: 25 parts, among them U1 TPS63001DRCT

Commit message: Finished WeBee
Parts:
- removed C12, C8: 10uF, rcl:C-EUC0603
- removed J1: (no value), SparkFun-Connectors:JST_2MM_MALE
- removed L2: 2.2uH, SparkFun-Passives:INDUCTOR0805
- removed U1: TPS63001DRCT, TPS63001:TPS63001DRCT
- added C4, C5: 22uF, rcl:C-EUC0603
- added C7: 0.1uF, adafruit:C-USC0402
- added D3: BAT20J, SparkFun-DiscreteSemi:DIODE-SCHOTTKY-BAT20J
- added J2: (no value), SparkFun-Connectors:JST_2MM_MALE
- added L1: 2.2uH, Spark:INDUCTOR-SPARKFUN0805
- added R16: 10K 1%, SparkFun-Resistors:RESISTOR0603
- added R3: 0, SparkFun-Passives:RESISTOR0603-RES
- added R4: 100K, adafruit:R-US_R0402
- added R5: (no value), microbuilder:RESISTOR0402
- added R8: 45.2k 1%, SparkFun-Resistors:RESISTOR0603
- added S1: (no value), Spark:TAC_SWITCHSMD
- added U3: LMR10510XMFE, Microchip_By_element14_Batch_1:LMR10510XMFE
Connections:
- removed net N$65: L2.1, U1.L1
- removed net N$66: L2.2, U1.L2
- new net FB: R16.2, R8.1, U3.FB
- new net N$1: R5.1, S1.2
- new net N$11: R4.1, U3.EN
- new net SW: D3.C, L1.1, U3.SW
- net +5V_USB: now also R3.2
- net +BATT: now also J2.+; no longer J1.+
- net GND: now also C4.2, C5.2, C7.2, D3.A, J2.-, R16.1, S1.3, S1.4, U3.GND; no longer C12.2, C8.2, J1.-, U1.GND, U1.PGND, U1.POWER_PAD
- net OUT: now also C4.1, R3.1, R4.2, U3.VIN; no longer C12.1, U1.EN, U1.PS/SYNC, U1.VIN, U1.VINA
- net VCC: now also C5.1, C7.1, L1.2, R5.2, R8.2; no longer C8.1, U1.FB, U1.VOUT
Other:
- note removed: "3.3V"
- note removed: "BATT"
- note removed: "Optional"
- note removed: "Voltage Regulator"
