File: Breakout/FTDI Only/ftdi.brd (EAGLE design)
At the start: 19.4 x 22.8 mm, 28 parts, among them Q1 16Mhz, U5 93LC46BT-I/OT

Commit message: ftdi changes
Parts:
- removed Q1: 16Mhz, crystal:TC26H
- removed U$3: DECADE-74LVC125A, DECADE-libraries:DECADE-SO-14
- added U1: SN74LVC126APW, Texas Instruments_By_element14_Batch_1:SOP65P640X120-14N
- added U2, U3: SN74LVC125APW, Texas Instruments_By_element14_Batch_1:SOP65P640X120-14N
- added Y1: 6Mhz, microbuilder:CRYSTAL_2.5X2
- moved R10 21.8 mm to (29.4, 2.40)
- moved R9 21.2 mm to (29.3, 4.60)
Connections:
- net DBGEN_N: no longer U$3.1
- net DBG_RST_N: no longer U$3.4
- net FT_SK: no longer U$3.2
- net GND: no longer U$3.7
- net N$38: now also Y1.3; no longer Q1.2
- net N$40: now also Y1.1; no longer Q1.1
- net N$49: no longer U$3.5
- net N$50: no longer U$3.6
- net TCK: no longer U$3.3
- net VCC: now also U1.14, U2.14, U3.14; no longer U$3.14
Other:
- board size 19.4 x 22.8 mm -> 19.4 x 28.6 mm
