File: Breakout/FTDI Only/ftdi.sch (EAGLE design)
At the start: 28 parts, among them Q1 16Mhz, U5 93LC46BT-I/OT

Commit message: ftdi changes
Parts:
- removed Q1: 16Mhz, crystal:CRYSTALTC26H
- removed U$3: DECADE-74LVC125A, DECADE-libraries:DECADE-74LVC125A
- added U1: SN74LVC126APW, Texas Instruments_By_element14_Batch_1:SN74LVC126APW
- added U2, U3: SN74LVC125APW, Texas Instruments_By_element14_Batch_1:SN74LVC125APW
- added Y1: 6Mhz, microbuilder:CRYSTAL2.5X2.0MM
Connections:
- net DBGEN_N: no longer U$3.OE1
- net DBG_RST_N: no longer U$3.OE2
- net FT_SK: no longer U$3.1A
- net GND: no longer U$3.GND
- net N$38: now also Y1.2; no longer Q1.2
- net N$40: now also Y1.1; no longer Q1.1
- net N$49: no longer U$3.2A
- net N$50: no longer U$3.2Y
- net TCK: no longer U$3.1Y
- net VCC: no longer U$3.VCC
Changed lines of the file:
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@@
 <setting verticaltext="up"/>
 </settings>
-<grid distance="0.01" unitdist="inch" unit="inch" style="lines" multiple="1" display="no" altdistance="0.01" altunitdist="inch" altunit="inch"/>
+<grid distance="0.1" unitdist="inch" unit="inch" style="lines" multiple="1" display="no" altdistance="0.01" altunitdist="inch" altunit="inch"/>
 <layers>
 <layer number="1" name="Top" color="4" fill="1" visible="no" active="no"/>
@@
 <part name="FRAME1" library="frames" deviceset="FRAME_D_L" device=""/>
 <part name="U$1" library="SparkFun-DigitalIC" deviceset="FT2232D" device=""/>
-<part name="Q1" library="crystal" deviceset="CRYSTAL" device="TC26H" value="16Mhz"/>
 <part name="C2" library="SparkFun-Passives" deviceset="CAP" device="0402-CAP" value="27pF"/>
 <part name="C3" library="SparkFun-Passives" deviceset="CAP" device="0402-CAP" value="27pF"/>
 <part name="C4" library="SparkFun-Passives" deviceset="CAP" device="0402-CAP" value="33nF"/>
-<part name="U$3" library="DECADE-libraries" deviceset="DECADE-74LVC125A" device=""/>
 <part name="C5" library="SparkFun-Passives" deviceset="CAP" device="0402-CAP" value="0.1uF"/>
 <part name="L3" library="Spark" deviceset="INDUCTOR-SPARKFUN" device="0603"/>
@@
 <part name="R1" library="SparkFun-Passives" deviceset="RESISTOR" device="0402-RES" value="28"/>
 <part name="R15" library="SparkFun-Passives" deviceset="RESISTOR" device="0402-RES" value="28"/>
+<part name="U1" library="Texas Instruments_By_element14_Batch_1" deviceset="SN74LVC126APW" device=""/>
+<part name="U2" library="Texas Instruments_By_element14_Batch_1" deviceset="SN74LVC125APW" device=""/>
+<part name="U3" library="Texas Instruments_By_element14_Batch_1" deviceset="SN74LVC125APW" device=""/>
+<part name="Y1" library="microbuilder" deviceset="CRYSTAL" device="2.5X2.0MM" value="6Mhz"/>
 </parts>
 <sheets>
@@
 <instance part="FRAME1" gate="G$2" x="755.65" y="-2.54"/>
 <instance part="U$1" gate="G$1" x="124.46" y="317.5"/>
-<instance part="Q1" gate="G$1" x="63.5" y="317.5" rot="R90"/>
 <instance part="C2" gate="G$1" x="55.88" y="322.58" rot="R90"/>
 <instance part="C3" gate="G$1" x="55.88" y="309.88" rot="R90"/>
 <instance part="C4" gate="G$1" x="88.9" y="342.9" rot="R90"/>
-<instance part="U$3" gate="G$1" x="234.95" y="317.5"/>
 <instance part="C5" gate="G$1" x="68.58" y="355.6" rot="R90"/>
 <instance part="L3" gate="G$1" x="48.26" y="340.36" rot="R90"/>
@@
 <attribute name="VALUE" x="55.88" y="350.012" size="1.778" layer="96" rot="R180"/>
 </instance>
+<instance part="U1" gate="A" x="332.74" y="325.12"/>
+<instance part="U2" gate="A" x="335.28" y="271.78"/>
+<instance part="U3" gate="A" x="383.54" y="271.78"/>
+<instance part="Y1" gate="G$1" x="63.5" y="317.5" rot="R90"/>
 </instances>
 <busses>
@@
 </segment>
 <segment>
-<pinref part="U$3" gate="G$1" pin="GND"/>
 <wire x1="217.17" y1="304.8" x2="209.55" y2="304.8" width="0.1524" layer="91"/>
 <label x="203.2" y="306.07" size="1.778" layer="95"/>
@@
 <net name="VCC" class="0">
 <segment>
-<pinref part="U$3" gate="G$1" pin="VCC"/>
 <wire x1="276.86" y1="335.28" x2="287.02" y2="335.28" width="0.1524" layer="91"/>
 <label x="288.29" y="335.28" size="1.778" layer="95"/>
@@
 <net name="N$38" class="0">
 <segment>
-<pinref part="Q1" gate="G$1" pin="2"/>
 <wire x1="63.5" y1="320.04" x2="63.5" y2="322.58" width="0.1524" layer="91"/>
 <wire x1="63.5" y1="322.58" x2="71.12" y2="322.58" width="0.1524" layer="91"/>
@@
 <pinref part="C2" gate="G$1" pin="2"/>
 <wire x1="58.42" y1="322.58" x2="63.5" y2="322.58" width="0.1524" layer="91"/>
+<pinref part="Y1" gate="G$1" pin="2"/>
 </segment>
 </net>
@@
 <wire x1="104.14" y1="314.96" x2="71.12" y2="314.96" width="0.1524" layer="91"/>
 <wire x1="71.12" y1="314.96" x2="71.12" y2="309.88" width="0.1524" layer="91"/>
-<pinref part="Q1" gate="G$1" pin="1"/>
 <wire x1="71.12" y1="309.88" x2="63.5" y2="309.88" width="0.1524" layer="91"/>
 <wire x1="63.5" y1="309.88" x2="63.5" y2="314.96" width="0.1524" layer="91"/>
 <pinref part="C3" gate="G$1" pin="2"/>
 <wire x1="58.42" y1="309.88" x2="63.5" y2="309.88" width="0.1524" layer="91"/>
+<pinref part="Y1" gate="G$1" pin="1"/>
 </segment>
 </net>
@@
 <net name="TCK" class="0">
 <segment>
-<pinref part="U$3" gate="G$1" pin="1Y"/>
 <wire x1="217.17" y1="325.12" x2="212.09" y2="325.12" width="0.1524" layer="91"/>
 <label x="210.82" y="322.58" size="1.778" layer="95"/>
@@
 <net name="DBGEN_N" class="0">
 <segment>
-<pinref part="U$3" gate="G$1" pin="OE1"/>
 <label x="199.39" y="335.28" size="1.778" layer="95"/>
 <wire x1="161.29" y1="340.36" x2="166.37" y2="340.36" width="0.1524" layer="91"/>
@@
 <net name="FT_SK" class="0">
 <segment>
-<pinref part="U$3" gate="G$1" pin="1A"/>
 <label x="203.2" y="330.2" size="1.778" layer="95"/>
 <wire x1="161.29" y1="355.6" x2="171.45" y2="355.6" width="0.1524" layer="91"/>
@@
 <wire x1="179.07" y1="342.9" x2="179.07" y2="346.71" width="0.1524" layer="91"/>
 <wire x1="179.07" y1="342.9" x2="179.07" y2="320.04" width="0.1524" layer="91"/>
-<pinref part="U$3" gate="G$1" pin="OE2"/>
 <wire x1="179.07" y1="320.04" x2="217.17" y2="320.04" width="0.1524" layer="91"/>
 <label x="181.61" y="342.9" size="1.778" layer="95"/>
@@
 <net name="N$49" class="0">
 <segment>
-<pinref part="U$3" gate="G$1" pin="2A"/>
 <wire x1="212.09" y1="314.96" x2="217.17" y2="314.96" width="0.1524" layer="91"/>
 <pinref part="R10" gate="G$1" pin="1"/>
@@
 <net name="N$50" class="0">
 <segment>
-<pinref part="U$3" gate="G$1" pin="2Y"/>
 <wire x1="212.09" y1="309.88" x2="217.17" y2="309.88" width="0.1524" layer="91"/>
 <pinref part="R9" gate="G$1" pin="1"/>
